File: kiss-masterboard/masterboard_v0.2/Sensors.kicad_sch (KiCad schematic)
At the start: 8 parts, among them U15 MPU-9250, U16 ADS1000

Commit message: replaced symbosl with standart symbols and reduced DRC errorsMAX98357A and TLV75709PDBV symbols
Parts:
- removed C66: 10nF, Capacitor_SMD:C_0603_1608Metric, symbol Device:C
- removed C67, C68, C69: 100nF, Capacitor_SMD:C_0603_1608Metric, symbol Device:C
- removed R49: 10K 1%, Resistor_SMD:R_0603_1608Metric, symbol Device:R
- removed R50: 1.78K 1%, Resistor_SMD:R_0603_1608Metric, symbol Device:R
- removed U15: MPU-9250, Sensor_Motion:InvenSense_QFN-24_3x3mm_P0.4mm, symbol Sensor_Motion:MPU-9250
- removed U16: ADS1000, Package_TO_SOT_SMD:SOT-23-6, symbol Power_Board:ADS1000
Connections:
- no-connect marks 5 -> 0
Other:
- note removed: "AD Wandler"
- note removed: "IMU"
