File: kiss-masterboard/masterboard_v0.2/PanelPower.kicad_sch (KiCad schematic)
At the start: 27 parts, among them U10 CSD86360Q5D, U9 TPS53819A

Commit message: Add extension header
Parts:
- removed C46, C48, C50, C52: 47µF, Power_Board:CP_OSCON_Poly_F12, symbol Device:C_Polarized
- removed C47, C49, C51: 47µF, Capacitor_SMD:C_1210_3225Metric, symbol Device:C
- added C46, C48, C50, C52, C55, C59, C60, C62: 22uF, Capacitor_SMD:C_1206_3216Metric, symbol Device:C
- added C63, C64, C65: 47uF, Capacitor_SMD:C_1206_3216Metric, symbol Device:C
- C53: value 47µF -> 47uF; footprint Capacitor_SMD:C_1210_3225Metric -> Capacitor_SMD:C_1206_3216Metric; Digikey No. 490-10531-1-ND -> (none); Manufacturer Murata -> (none); Part No. GRM32EC81C476KE15L -> C12891
Connections:
- net GND: now also C46.2, C48.2, C50.2, C52.2, C55.2, C59.2, C60.2, C62.2, C63.2, C64.2, C65.2
- net Panel_Power: now also C63.1, C64.1, C65.1
- net Power_in: now also C46.1, C48.1, C50.1, C52.1, C55.1, C59.1, C60.1, C62.1

Commit message: Added IMU, routed extension layer, switched battery polarity
Parts:
- C39, C40: value 1µF -> 1uF
- C43, C44, C45: value 10µF -> 10uF
- R36: value 38.3K -> 38.3k
- R37: value 294K -> 294k
- R39: value 100K -> 100k
Changed lines of the file:
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@@
 			)
 		)
-		(property "Value" "1µF"
+		(property "Value" "1uF"
 			(at 60.96 50.8 0)
 			(show_name no)
@@
 			)
 		)
-		(property "Value" "100K"
+		(property "Value" "100k"
 			(at 83.058 49.403 0)
 			(show_name no)
@@
 			)
 		)
-		(property "Value" "294K"
+		(property "Value" "294k"
 			(at 70.358 49.403 0)
 			(show_name no)
@@
 			)
 		)
-		(property "Value" "38.3K"
+		(property "Value" "38.3k"
 			(at 52.578 128.143 0)
 			(show_name no)
@@
 			)
 		)
-		(property "Value" "1µF"
+		(property "Value" "1uF"
 			(at 43.18 50.8 0)
 			(show_name no)
@@
 			)
 		)
-		(property "Value" "10µF"
+		(property "Value" "10uF"
 			(at 220.98 73.66 0)
 			(show_name no)
@@
 			)
 		)
-		(property "Value" "10µF"
+		(property "Value" "10uF"
 			(at 220.98 43.18 0)
 			(show_name no)
@@
 			)
 		)
-		(property "Value" "10µF"
+		(property "Value" "10uF"
 			(at 212.09 43.18 0)
 			(show_name no)

Commit message: add cnumbers initial order v04a
Parts:
- C39: JLCNR (none) -> C28323
- C40: JLCNR (none) -> C15849
- C41: JLCNR (none) -> C49678
- C42: JLCNR (none) -> C1588
- C43, C44, C45: JLCNR (none) -> C13585
- C46, C48, C50, C52, C55, C59, C60, C62: JLCNR (none) -> C12891
- C53, C63, C64, C65: JLCNR (none) -> C96123
- L1: JLCNR (none) -> C3911594
- R36: JLCNR (none) -> C2999480
- R37: JLCNR (none) -> C3013161
- R38: JLCNR (none) -> C11710
- R39: JLCNR (none) -> C25803
- R40, R42: JLCNR (none) -> C25271
- R41: JLCNR (none) -> C17675
- R43: JLCNR (none) -> C25804
- R44: JLCNR (none) -> C861207
- U10: JLCNR (none) -> C181654; now not fitted
- U9: JLCNR (none) -> C702272; now not fitted
