File: kiss-masterboard/masterboard_v0.2/PanelPower.kicad_sch (KiCad schematic)
At the start: 31 parts, among them U10 CSD86360Q5D, U9 TPS53819A

Commit message: adjust c numbers and footprint for hab75
Parts:
- C39: JLCNR C28323 -> (none); LCSC Part # (none) -> C28323
- C40: JLCNR C15849 -> (none); LCSC Part # (none) -> C15849
- C41: JLCNR C49678 -> (none); LCSC Part # (none) -> C49678
- C42: JLCNR C1588 -> (none); LCSC Part # (none) -> C1588
- C43, C44, C45: JLCNR C13585 -> (none); LCSC Part # (none) -> C13585
- C46, C48, C50, C52, C55, C59, C60, C62: JLCNR C12891 -> (none); LCSC Part # (none) -> C12891
- C53, C63, C64, C65: JLCNR C96123 -> (none); LCSC Part # (none) -> C96123
- L1: JLCNR C3911594 -> (none); LCSC Part # (none) -> C3911594
- R36: JLCNR C2999480 -> (none); LCSC Part # (none) -> C2999480
- R37: JLCNR C3013161 -> (none); LCSC Part # (none) -> C3013161
- R38: JLCNR C11710 -> (none); LCSC Part # (none) -> C11710
- R39: JLCNR C25803 -> (none); LCSC Part # (none) -> C25803
- R40, R42: JLCNR C25271 -> (none); LCSC Part # (none) -> C25271
- R41: JLCNR C17675 -> (none); LCSC Part # (none) -> C17675
- R43: JLCNR C25804 -> (none); LCSC Part # (none) -> C25804
- R44: JLCNR C861207 -> (none); LCSC Part # (none) -> C861207
- U10: JLCNR C181654 -> (none); LCSC Part # (none) -> C181654
- U9: JLCNR C702272 -> (none); LCSC Part # (none) -> C702272
Changed lines of the file:
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@@
 			)
 		)
-		(property "JLCNR" "C15849"
+		(property "LCSC Part #" "C15849"
 			(at 59.69 48.26 0)
 			(hide yes)
@@
 			)
 		)
-		(property "JLCNR" "C25803"
+		(property "LCSC Part #" "C25803"
 			(at 81.28 48.26 0)
 			(hide yes)
@@
 			)
 		)
-		(property "JLCNR" "C3013161"
+		(property "LCSC Part #" "C3013161"
 			(at 68.58 48.26 0)
 			(hide yes)
@@
 			)
 		)
-		(property "JLCNR" "C11710"
+		(property "LCSC Part #" "C11710"
 			(at 68.58 63.5 0)
 			(hide yes)
@@
 			)
 		)
-		(property "JLCNR" "C702272"
+		(property "LCSC Part #" "C702272"
 			(at 81.28 101.6 0)
 			(hide yes)
@@
 			)
 		)
-		(property "JLCNR" "C2999480"
+		(property "LCSC Part #" "C2999480"
 			(at 50.8 127 0)
 			(hide yes)
@@
 			)
 		)
-		(property "JLCNR" "C17675"
+		(property "LCSC Part #" "C17675"
 			(at 123.19 97.79 90)
 			(hide yes)
@@
 			)
 		)
-		(property "JLCNR" "C49678"
+		(property "LCSC Part #" "C49678"
 			(at 123.19 86.36 90)
 			(hide yes)
@@
 			)
 		)
-		(property "JLCNR" "C25271"
+		(property "LCSC Part #" "C25271"
 			(at 111.76 86.36 90)
 			(hide yes)
@@
 			)
 		)
-		(property "JLCNR" "C28323"
+		(property "LCSC Part #" "C28323"
 			(at 41.91 48.26 0)
 			(hide yes)
@@
 			)
 		)
-		(property "JLCNR" "C13585"
+		(property "LCSC Part #" "C13585"
 			(at 219.71 71.12 0)
 			(hide yes)
@@
 			)
 		)
-		(property "JLCNR" "C861207"
+		(property "LCSC Part #" "C861207"
 			(at 181.61 123.19 0)
 			(hide yes)
@@
 			)
 		)
-		(property "JLCNR" "C25804"
+		(property "LCSC Part #" "C25804"
 			(at 181.61 110.49 0)
 			(hide yes)
@@
 			)
 		)
-		(property "JLCNR" "C1588"
+		(property "LCSC Part #" "C1588"
 			(at 163.83 110.49 0)
 			(hide yes)
@@
 			)
 		)
-		(property "JLCNR" "C25271"
+		(property "LCSC Part #" "C25271"
 			(at 163.83 123.19 0)
 			(hide yes)
@@
 			)
 		)
-		(property "JLCNR" "C3911594"
+		(property "LCSC Part #" "C3911594"
 			(at 172.72 102.87 90)
 			(hide yes)
@@
 			)
 		)
-		(property "JLCNR" "C181654"
+		(property "LCSC Part #" "C181654"
 			(at 144.78 101.6 0)
 			(hide yes)
@@
 			)
 		)
-		(property "JLCNR" "C13585"
+		(property "LCSC Part #" "C13585"
 			(at 219.71 40.64 0)
 			(hide yes)
@@
 			)
 		)
-		(property "JLCNR" "C13585"
+		(property "LCSC Part #" "C13585"
 			(at 210.82 40.64 0)
 			(hide yes)
@@
 			)
 		)
-		(property "JLCNR" "C12891"
+		(property "LCSC Part #" "C12891"
 			(at 260.35 40.64 0)
 			(hide yes)
@@
 			)
 		)
-		(property "JLCNR" "C96123"
+		(property "LCSC Part #" "C96123"
 			(at 260.35 71.12 0)
 			(hide yes)
@@
 			)
 		)
-		(property "JLCNR" "C96123"
+		(property "LCSC Part #" "C96123"
 			(at 240.03 71.12 0)
 			(hide yes)
@@
 			)
 		)
-		(property "JLCNR" "C12891"
+		(property "LCSC Part #" "C12891"
 			(at 250.19 40.64 0)
 			(hide yes)
@@
 			)
 		)
-		(property "JLCNR" "C12891"
+		(property "LCSC Part #" "C12891"
 			(at 234.95 40.64 0)
 			(hide yes)
@@
 			)
 		)
-		(property "JLCNR" "C12891"
+		(property "LCSC Part #" "C12891"
 			(at 255.27 40.64 0)
 			(hide yes)
@@
 			)
 		)
-		(property "JLCNR" "C12891"
+		(property "LCSC Part #" "C12891"
 			(at 245.11 40.64 0)
 			(hide yes)
@@
 			)
 		)
-		(property "JLCNR" "C96123"
+		(property "LCSC Part #" "C96123"
 			(at 250.19 71.12 0)
 			(hide yes)
@@
 			)
 		)
-		(property "JLCNR" "C96123"
+		(property "LCSC Part #" "C96123"
 			(at 229.87 71.12 0)
 			(hide yes)
@@
 			)
 		)
-		(property "JLCNR" "C12891"
+		(property "LCSC Part #" "C12891"
 			(at 224.79 40.64 0)
 			(hide yes)
@@
 			)
 		)
-		(property "JLCNR" "C12891"
+		(property "LCSC Part #" "C12891"
 			(at 229.87 40.64 0)
 			(hide yes)
@@
 			)
 		)
-		(property "JLCNR" "C12891"
+		(property "LCSC Part #" "C12891"
 			(at 240.03 40.64 0)
 			(hide yes)
