File: kiss-masterboard/masterboard_v0.2/DigitalAudio.kicad_sch (KiCad schematic)
At the start: 5 parts, among them U7 SPH0645LM4H

Commit message: adjust c numbers and footprint for hab75
Parts:
- C35: JLCNR C15849 -> (none); LCSC Part # (none) -> C15849
- C36: JLCNR C1603 -> (none); LCSC Part # (none) -> C1603
- R34: JLCNR C25804 -> (none); LCSC Part # (none) -> C25804
- R35: JLCNR C27592 -> (none); LCSC Part # (none) -> C27592
Changed lines of the file:
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@@
-			)
-		)
-		(property "JLCNR" ""
-			(at 80.01 86.36 0)
-			(hide yes)
-			(show_name no)
-			(do_not_autoplace no)
-			(effects
-				(font
-					(size 3.9878 3.9878)
-				)
 			)
 		)
@@
 			)
 		)
-		(property "JLCNR" "C25804"
+		(property "LCSC Part #" "C25804"
 			(at 66.04 93.98 0)
 			(hide yes)
@@
 			)
 		)
-		(property "JLCNR" "C27592"
+		(property "LCSC Part #" "C27592"
 			(at 101.6 86.36 90)
 			(hide yes)
@@
 			)
 		)
-		(property "JLCNR" "C15849"
+		(property "LCSC Part #" "C15849"
 			(at 45.72 92.71 0)
 			(hide yes)
@@
 			)
 		)
-		(property "JLCNR" "C1603"
+		(property "LCSC Part #" "C1603"
 			(at 52.07 92.71 0)
 			(hide yes)
