File: kiss-masterboard/masterboard_v0.2/Raspi.kicad_sch (KiCad schematic)
At the start: 3 parts, among them P2 CONN_02X20

Commit message: adjust c numbers and footprint for hab75
Parts:
- P2: JLCNR C22436166 -> (none); LCSC Part # (none) -> C22436166
- R31, R32: JLCNR C25803 -> (none); LCSC Part # (none) -> C25803
Changed lines of the file:
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@@
 			)
 		)
-		(property "JLCNR" "C25803"
+		(property "LCSC Part #" "C25803"
 			(at 92.71 48.26 90)
 			(hide yes)
@@
 			)
 		)
-		(property "JLCNR" "C25803"
+		(property "LCSC Part #" "C25803"
 			(at 97.79 48.26 90)
 			(hide yes)
@@
 			)
 		)
-		(property "JLCNR" "C22436166"
+		(property "LCSC Part #" "C22436166"
 			(at 49.53 52.07 0)
 			(hide yes)
