File: kiss-masterboard/masterboard_v0.2/RaspiPower.kicad_sch (KiCad schematic)
At the start: 13 parts, among them U3 TPS56339DDC

Commit message: adjust c numbers and footprint for hab75
Parts:
- C1, C2: JLCNR C440198 -> (none); LCSC Part # (none) -> C440198
- C32, C5: JLCNR C14663 -> (none); LCSC Part # (none) -> C14663
- C58, C7: JLCNR C12891 -> (none); LCSC Part # (none) -> C12891
- L8: JLCNR C3040411 -> (none); LCSC Part # (none) -> C3040411
- R10: JLCNR C2930115 -> (none); LCSC Part # (none) -> C2930115
- R11: JLCNR C25804 -> (none); LCSC Part # (none) -> C25804
- R12: JLCNR C23231 -> (none); LCSC Part # (none) -> C23231
- R13: JLCNR C5159703 -> (none); LCSC Part # (none) -> C5159703
- R9: JLCNR C217958 -> (none); LCSC Part # (none) -> C217958
- U3: JLCNR C2071106 -> (none); LCSC Part # (none) -> C2071106
Changed lines of the file:
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@@
 			)
 		)
-		(property "JLCNR" "C14663"
+		(property "LCSC Part #" "C14663"
 			(at 49.53 40.64 0)
 			(hide yes)
@@
 			)
 		)
-		(property "JLCNR" " C440198"
+		(property "LCSC Part #" " C440198"
 			(at 34.29 40.64 0)
 			(hide yes)
@@
 			)
 		)
-		(property "JLCNR" "C14663"
+		(property "LCSC Part #" "C14663"
 			(at 110.49 40.64 90)
 			(hide yes)
@@
 			)
 		)
-		(property "JLCNR" "C3040411"
+		(property "LCSC Part #" "C3040411"
 			(at 121.92 34.29 90)
 			(hide yes)
@@
 			)
 		)
-		(property "JLCNR" "C2930115"
+		(property "LCSC Part #" "C2930115"
 			(at 129.54 39.37 0)
 			(hide yes)
@@
 			)
 		)
-		(property "JLCNR" "C25804"
+		(property "LCSC Part #" "C25804"
 			(at 129.54 49.53 0)
 			(hide yes)
@@
 			)
 		)
-		(property "JLCNR" "C12891"
+		(property "LCSC Part #" "C12891"
 			(at 140.97 44.45 0)
 			(hide yes)
@@
 			)
 		)
-		(property "JLCNR" "C12891"
+		(property "LCSC Part #" "C12891"
 			(at 148.59 44.45 0)
 			(hide yes)
@@
 			)
 		)
-		(property "JLCNR" " C440198"
+		(property "LCSC Part #" " C440198"
 			(at 41.91 40.64 0)
 			(hide yes)
@@
 			)
 		)
-		(property "JLCNR" "C5159703"
+		(property "LCSC Part #" "C5159703"
 			(at 72.39 44.45 90)
 			(hide yes)
@@
 			)
 		)
-		(property "JLCNR" "C23231"
+		(property "LCSC Part #" "C23231"
 			(at 68.58 44.45 90)
 			(hide yes)
@@
 			)
 		)
-		(property "JLCNR" "C217958"
+		(property "LCSC Part #" "C217958"
 			(at 101.6 40.64 90)
 			(hide yes)
@@
 			)
 		)
-		(property "JLCNR" "C2071106"
+		(property "LCSC Part #" "C2071106"
 			(at 83.82 34.29 0)
 			(hide yes)
