File: kiss-masterboard/masterboard_v0.2/kiss-masterboard.kicad_sch (KiCad schematic)
At the start: 31 parts, among them J1 Cubebatt_host, J17 Conn_02x05_Counter_Clockwise, J18 Conn_02x02_Counter_Clockwise, J2 Conn_01x02, J3 Conn_01x02, J4 Conn_01x02, J5 Conn_01x02, J6 Conn_01x02, J7 Conn_01x02, J9 Conn_01x07_Pin

Commit message: adjust c numbers and footprint for hab75
Parts:
- D1: JLCNR C2290 -> (none); LCSC Part # (none) -> C2290
- D2: JLCNR C2286 -> (none); LCSC Part # (none) -> C2286
- D3: JLCNR C5818966 -> (none); LCSC Part # (none) -> C5818966
- J17: value Conn_02x05_Counter_Clockwise -> Conn_02x06_Counter_Clockwise; JLCNR C32713285 -> (none); LCSC Part # (none) -> C32713286
- J18: JLCNR C919361 -> (none); LCSC Part # (none) -> C919361
- L2, L3, L4, L5, L6, L7: JLCNR C48543410 -> (none); LCSC Part # (none) -> C48543410
- R1, R2, R3, R6, R7, R8: JLCNR C21189 -> (none); LCSC Part # (none) -> C21189
- R4, R5: JLCNR C23228 -> (none); LCSC Part # (none) -> C23228
Changed lines of the file:
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@@
 			)
 		)
-		(property "JLCNR" "C23228"
+		(property "LCSC Part #" "C23228"
 			(at 48.26 170.18 0)
 			(hide yes)
@@
 			)
 		)
-		(property "JLCNR" "C2286"
+		(property "LCSC Part #" "C2286"
 			(at 48.26 157.48 90)
 			(hide yes)
@@
 			)
 		)
-		(property "JLCNR" "C48543410"
+		(property "LCSC Part #" "C48543410"
 			(at 245.11 24.13 90)
 			(hide yes)
@@
 			)
 		)
-		(property "JLCNR" "C48543410"
+		(property "LCSC Part #" "C48543410"
 			(at 245.11 31.75 90)
 			(hide yes)
@@
 			)
 		)
-		(property "JLCNR" "C48543410"
+		(property "LCSC Part #" "C48543410"
 			(at 245.11 39.37 90)
 			(hide yes)
@@
 			)
 		)
-		(property "JLCNR" "C48543410"
+		(property "LCSC Part #" "C48543410"
 			(at 245.11 46.99 90)
 			(hide yes)
@@
 			)
 		)
-		(property "JLCNR" "C48543410"
+		(property "LCSC Part #" "C48543410"
 			(at 245.11 54.61 90)
 			(hide yes)
@@
 			)
 		)
-		(property "JLCNR" "C48543410"
+		(property "LCSC Part #" "C48543410"
 			(at 245.11 62.23 90)
 			(hide yes)
@@
 			)
 		)
-		(property "JLCNR" "C23228"
+		(property "LCSC Part #" "C23228"
 			(at 38.1 170.18 0)
 			(hide yes)
@@
 			)
 		)
-		(property "JLCNR" "C2290"
+		(property "LCSC Part #" "C2290"
 			(at 38.1 157.48 90)
 			(hide yes)
@@
 			)
 		)
-		(property "JLCNR" ""
-			(at 264.16 151.13 0)
-			(hide yes)
-			(show_name no)
-			(do_not_autoplace no)
-			(effects
-				(font
-					(size 3.9878 3.9878)
-				)
-			)
-		)
 		(instances
 			(project "kiss-masterboard"
@@
 			)
 		)
-		(property "JLCNR" ""
-			(at 264.16 138.43 0)
-			(hide yes)
-			(show_name no)
-			(do_not_autoplace no)
-			(effects
-				(font
-					(size 3.9878 3.9878)
-				)
-			)
-		)
 		(instances
 			(project "kiss-masterboard"
@@
 			)
 		)
-		(property "JLCNR" ""
-			(at 264.16 158.75 0)
-			(hide yes)
-			(show_name no)
-			(do_not_autoplace no)
-			(effects
-				(font
-					(size 3.9878 3.9878)
-				)
-			)
-		)
 		(instances
 			(project "kiss-masterboard"
@@
 			)
 		)
-		(property "JLCNR" ""
-			(at 29.21 31.75 0)
-			(hide yes)
-			(show_name no)
-			(do_not_autoplace no)
-			(effects
-				(font
-					(size 3.9878 3.9878)
-				)
-			)
-		)
 		(pin "1"
 		)
@@
 			)
 		)
-		(property "JLCNR" "C21189"
+		(property "LCSC Part #" "C21189"
 			(at 38.1 27.94 90)
 			(hide yes)
@@
 			)
 		)
-		(property "JLCNR" "C21189"
+		(property "LCSC Part #" "C21189"
 			(at 38.1 30.48 90)
 			(hide yes)
@@
 			)
 		)
-		(property "JLCNR" "C21189"
+		(property "LCSC Part #" "C21189"
 			(at 38.1 33.02 90)
 			(hide yes)
@@
 			)
 		)
-		(property "JLCNR" "C21189"
+		(property "LCSC Part #" "C21189"
 			(at 158.75 38.1 90)
 			(hide yes)
@@
 			)
 		)
-		(property "JLCNR" "C21189"
+		(property "LCSC Part #" "C21189"
 			(at 158.75 40.64 90)
 			(hide yes)
@@
 			)
 		)
-		(property "JLCNR" ""
-			(at 261.62 24.13 0)
-			(hide yes)
-			(show_name no)
-			(do_not_autoplace no)
-			(effects
-				(font
-					(size 3.9878 3.9878)
-				)
-			)
-		)
 		(pin "1"
 		)
@@
 			)
 		)
-		(property "JLCNR" ""
-			(at 261.62 31.75 0)
-			(hide yes)
-			(show_name no)
-			(do_not_autoplace no)
-			(effects
-				(font
-					(size 3.9878 3.9878)
-				)
-			)
-		)
 		(pin "1"
 		)
@@
 			)
 		)
-		(property "JLCNR" ""
-			(at 261.62 39.37 0)
-			(hide yes)
-			(show_name no)
-			(do_not_autoplace no)
-			(effects
-				(font
-					(size 3.9878 3.9878)
-				)
-			)
-		)
 		(pin "1"
 		)
@@
 			)
 		)
-		(property "JLCNR" ""
-			(at 261.62 46.99 0)
-			(hide yes)
-			(show_name no)
-			(do_not_autoplace no)
-			(effects
-				(font
-					(size 3.9878 3.9878)
-				)
-			)
-		)
 		(pin "1"
 		)
@@
 			)
 		)
-		(property "JLCNR" ""
-			(at 261.62 54.61 0)
-			(hide yes)
-			(show_name no)
-			(do_not_autoplace no)
-			(effects
-				(font
-					(size 3.9878 3.9878)
-				)
-			)
-		)
 		(pin "1"
 		)
@@
 			)
 		)
-		(property "JLCNR" ""
-			(at 261.62 62.23 0)
-			(hide yes)
-			(show_name no)
-			(do_not_autoplace no)
-			(effects
-				(font
-					(size 3.9878 3.9878)
-				)
-			)
-		)
 		(pin "1"
 		)
@@
 			)
 		)
-		(property "JLCNR" "C21189"
+		(property "LCSC Part #" "C21189"
 			(at 38.1 35.56 90)
 			(hide yes)
@@
 			)
 		)
-		(property "JLCNR" ""
-			(at 17.78 19.05 0)
-			(hide yes)
-			(show_name no)
-			(do_not_autoplace no)
-			(effects
-				(font
-					(size 3.9878 3.9878)
-				)
-			)
-		)
 		(pin "1"
 		)
@@
 			)
 		)
-		(property "JLCNR" "C5818966"
+		(property "LCSC Part #" "C5818966"
 			(at 26.67 16.51 0)
 			(hide yes)
@@
 			)
 		)
-		(property "Value" "Conn_02x05_Counter_Clockwise"
+		(property "Value" "Conn_02x06_Counter_Clockwise"
 			(at 38.1 86.36 0)
 			(show_name no)
@@
 			)
 		)
-		(property "JLCNR" "C32713285"
+		(property "LCSC Part #" "C32713286"
 			(at 39.37 97.79 0)
 			(hide yes)
@@
 			)
 		)
-		(property "JLCNR" ""
-			(at 90.17 173.99 0)
-			(hide yes)
-			(show_name no)
-			(do_not_autoplace no)
-			(effects
-				(font
-					(size 3.9878 3.9878)
-				)
-			)
-		)
 		(pin "2"
 		)
@@
 			)
 		)
-		(property "JLCNR" "C919361"
+		(property "LCSC Part #" "C919361"
 			(at 36.83 80.01 0)
 			(hide yes)
