File: kiss-masterboard/masterboard_v0.2/kiss-masterboard.kicad_pcb (KiCad board)
At the start: 4 copper layers, 187 x 152 mm, 172 parts, among them J1 Cubebatt_host, J10 CRESET, J11 Jumper, J12 Jumper, J13 Conn_02x08_Odd_Even, J14 Conn_02x08_Odd_Even, J15 jmp, J16 jmp, J17 Conn_02x05_Counter_Clockwise, J18 Conn_02x02_Counter_Clockwise, J2 Conn_01x02, J3 Conn_01x02, J4 Conn_01x02, J5 Conn_01x02, J6 Conn_01x02, J7 Conn_01x02, J8 Jumper, J9 Conn_01x07_Pin, P2 CONN_02X20, U10 CSD86360Q5D, U11 TLV75733PDBV, U13 SN74LVC8T245, U14 W25Q, U17 12MHz, U2 SN74LVC8T245, U3 TPS56339DDC, U4 ICE40UP5k-SG48, U5 SN74LVC8T245, U7 SPH0645LM4H, U8 TLV75709PDBV, U9 TPS53819A

Commit message: kiss-masterboard: fix R51-R78 value, was 2.2M instead of 33E
R51-R78 (HUB75 LATCH/SCLK/BLANK/A0-A4/RGB data series resistors for
both panel connectors) were populated with 2-2.2M instead of the
intended 33E - a BOM/kitting error. 2.2M in series with these
CMOS-input lines low-pass filters the edges far too slowly for HUB75
timing at any usable clock, making the display unusable regardless of
gateware. Confirmed and hand-reworked on the physical board; corrected
here so the next fab run stuffs 33E instead of repeating the error.

Added a note next to the "Panel HUB75 Levelshifters" section
documenting this, and the related U17 (12MHz oscillator) fix.
Parts:
- R51, R52, R53, R54, R55, R56, R57, R58, R59, R60, R61, R62, R63, R64, R65, R66, R67, R68, R69, R70, R71, R72, R73, R74, R75, R76, R77, R78: value 2-2.2M (33E) -> 33E
Changed lines of the file:
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@@
 			)
 		)
-		(property "Value" "2-2.2M (33E)"
+		(property "Value" "33E"
 			(at 0 -1 0)
 			(layer "B.Fab")
@@
 			)
 		)
-		(property "Value" "2-2.2M (33E)"
+		(property "Value" "33E"
 			(at 0 -1 0)
 			(layer "B.Fab")
@@
 			)
 		)
-		(property "Value" "2-2.2M (33E)"
+		(property "Value" "33E"
 			(at 0 -1 0)
 			(layer "B.Fab")
@@
 			)
 		)
-		(property "Value" "2-2.2M (33E)"
+		(property "Value" "33E"
 			(at 0 -1 0)
 			(layer "B.Fab")
@@
 			)
 		)
-		(property "Value" "2-2.2M (33E)"
+		(property "Value" "33E"
 			(at 0 -1 0)
 			(layer "B.Fab")
@@
 			)
 		)
-		(property "Value" "2-2.2M (33E)"
+		(property "Value" "33E"
 			(at 0 -1 0)
 			(layer "B.Fab")
@@
 			)
 		)
-		(property "Value" "2-2.2M (33E)"
+		(property "Value" "33E"
 			(at 0 -1 0)
 			(layer "B.Fab")
@@
 			)
 		)
-		(property "Value" "2-2.2M (33E)"
+		(property "Value" "33E"
 			(at 0 -1 0)
 			(layer "B.Fab")
@@
 			)
 		)
-		(property "Value" "2-2.2M (33E)"
+		(property "Value" "33E"
 			(at 0 -1 0)
 			(layer "B.Fab")
@@
 			)
 		)
-		(property "Value" "2-2.2M (33E)"
+		(property "Value" "33E"
 			(at 0 -1 0)
 			(layer "B.Fab")
@@
 			)
 		)
-		(property "Value" "2-2.2M (33E)"
+		(property "Value" "33E"
 			(at 0 -1 0)
 			(layer "B.Fab")
@@
 			)
 		)
-		(property "Value" "2-2.2M (33E)"
+		(property "Value" "33E"
 			(at 0 -1 0)
 			(layer "B.Fab")
@@
 			)
 		)
-		(property "Value" "2-2.2M (33E)"
+		(property "Value" "33E"
 			(at 0 -1 0)
 			(layer "B.Fab")
@@
 			)
 		)
-		(property "Value" "2-2.2M (33E)"
+		(property "Value" "33E"
 			(at 0 -1 0)
 			(layer "B.Fab")
@@
 			)
 		)
-		(property "Value" "2-2.2M (33E)"
+		(property "Value" "33E"
 			(at 0 -1 0)
 			(layer "B.Fab")
@@
 			)
 		)
-		(property "Value" "2-2.2M (33E)"
+		(property "Value" "33E"
 			(at 0 -1 0)
 			(layer "B.Fab")
@@
 			)
 		)
-		(property "Value" "2-2.2M (33E)"
+		(property "Value" "33E"
 			(at 0 -1 0)
 			(layer "B.Fab")
@@
 			)
 		)
-		(property "Value" "2-2.2M (33E)"
+		(property "Value" "33E"
 			(at 0 -1 0)
 			(layer "B.Fab")
@@
 			)
 		)
-		(property "Value" "2-2.2M (33E)"
+		(property "Value" "33E"
 			(at 0 -1 0)
 			(layer "B.Fab")
@@
 			)
 		)
-		(property "Value" "2-2.2M (33E)"
+		(property "Value" "33E"
 			(at 0 -1 0)
 			(layer "B.Fab")
@@
 			)
 		)
-		(property "Value" "2-2.2M (33E)"
+		(property "Value" "33E"
 			(at 0 -1 0)
 			(layer "B.Fab")
@@
 			)
 		)
-		(property "Value" "2-2.2M (33E)"
+		(property "Value" "33E"
 			(at 0 -1 0)
 			(layer "B.Fab")
@@
 			)
 		)
-		(property "Value" "2-2.2M (33E)"
+		(property "Value" "33E"
 			(at 0 -1 0)
 			(layer "B.Fab")
@@
 			)
 		)
-		(property "Value" "2-2.2M (33E)"
+		(property "Value" "33E"
 			(at 0 -1 0)
 			(layer "B.Fab")
@@
 			)
 		)
-		(property "Value" "2-2.2M (33E)"
+		(property "Value" "33E"
 			(at 0 -1 0)
 			(layer "B.Fab")
@@
 			)
 		)
-		(property "Value" "2-2.2M (33E)"
+		(property "Value" "33E"
 			(at 0 -1 0)
 			(layer "B.Fab")
@@
 			)
 		)
-		(property "Value" "2-2.2M (33E)"
+		(property "Value" "33E"
 			(at 0 -1 0)
 			(layer "B.Fab")
@@
 			)
 		)
-		(property "Value" "2-2.2M (33E)"
+		(property "Value" "33E"
 			(at 0 -1 0)
 			(layer "B.Fab")

Commit message: Revert "kiss-masterboard: fix R51-R78 value, was 2.2M instead of 33E"
This reverts commit be2e0cd53d49abef9a9fc2547556a5b37668e0ac.
Parts:
- R51, R52, R53, R54, R55, R56, R57, R58, R59, R60, R61, R62, R63, R64, R65, R66, R67, R68, R69, R70, R71, R72, R73, R74, R75, R76, R77, R78: value 33E -> 2-2.2M (33E)
Changed lines of the file:
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@@
 			)
 		)
-		(property "Value" "33E"
+		(property "Value" "2-2.2M (33E)"
 			(at 0 -1 0)
 			(layer "B.Fab")
@@
 			)
 		)
-		(property "Value" "33E"
+		(property "Value" "2-2.2M (33E)"
 			(at 0 -1 0)
 			(layer "B.Fab")
@@
 			)
 		)
-		(property "Value" "33E"
+		(property "Value" "2-2.2M (33E)"
 			(at 0 -1 0)
 			(layer "B.Fab")
@@
 			)
 		)
-		(property "Value" "33E"
+		(property "Value" "2-2.2M (33E)"
 			(at 0 -1 0)
 			(layer "B.Fab")
@@
 			)
 		)
-		(property "Value" "33E"
+		(property "Value" "2-2.2M (33E)"
 			(at 0 -1 0)
 			(layer "B.Fab")
@@
 			)
 		)
-		(property "Value" "33E"
+		(property "Value" "2-2.2M (33E)"
 			(at 0 -1 0)
 			(layer "B.Fab")
@@
 			)
 		)
-		(property "Value" "33E"
+		(property "Value" "2-2.2M (33E)"
 			(at 0 -1 0)
 			(layer "B.Fab")
@@
 			)
 		)
-		(property "Value" "33E"
+		(property "Value" "2-2.2M (33E)"
 			(at 0 -1 0)
 			(layer "B.Fab")
@@
 			)
 		)
-		(property "Value" "33E"
+		(property "Value" "2-2.2M (33E)"
 			(at 0 -1 0)
 			(layer "B.Fab")
@@
 			)
 		)
-		(property "Value" "33E"
+		(property "Value" "2-2.2M (33E)"
 			(at 0 -1 0)
 			(layer "B.Fab")
@@
 			)
 		)
-		(property "Value" "33E"
+		(property "Value" "2-2.2M (33E)"
 			(at 0 -1 0)
 			(layer "B.Fab")
@@
 			)
 		)
-		(property "Value" "33E"
+		(property "Value" "2-2.2M (33E)"
 			(at 0 -1 0)
 			(layer "B.Fab")
@@
 			)
 		)
-		(property "Value" "33E"
+		(property "Value" "2-2.2M (33E)"
 			(at 0 -1 0)
 			(layer "B.Fab")
@@
 			)
 		)
-		(property "Value" "33E"
+		(property "Value" "2-2.2M (33E)"
 			(at 0 -1 0)
 			(layer "B.Fab")
@@
 			)
 		)
-		(property "Value" "33E"
+		(property "Value" "2-2.2M (33E)"
 			(at 0 -1 0)
 			(layer "B.Fab")
@@
 			)
 		)
-		(property "Value" "33E"
+		(property "Value" "2-2.2M (33E)"
 			(at 0 -1 0)
 			(layer "B.Fab")
@@
 			)
 		)
-		(property "Value" "33E"
+		(property "Value" "2-2.2M (33E)"
 			(at 0 -1 0)
 			(layer "B.Fab")
@@
 			)
 		)
-		(property "Value" "33E"
+		(property "Value" "2-2.2M (33E)"
 			(at 0 -1 0)
 			(layer "B.Fab")
@@
 			)
 		)
-		(property "Value" "33E"
+		(property "Value" "2-2.2M (33E)"
 			(at 0 -1 0)
 			(layer "B.Fab")
@@
 			)
 		)
-		(property "Value" "33E"
+		(property "Value" "2-2.2M (33E)"
 			(at 0 -1 0)
 			(layer "B.Fab")
@@
 			)
 		)
-		(property "Value" "33E"
+		(property "Value" "2-2.2M (33E)"
 			(at 0 -1 0)
 			(layer "B.Fab")
@@
 			)
 		)
-		(property "Value" "33E"
+		(property "Value" "2-2.2M (33E)"
 			(at 0 -1 0)
 			(layer "B.Fab")
@@
 			)
 		)
-		(property "Value" "33E"
+		(property "Value" "2-2.2M (33E)"
 			(at 0 -1 0)
 			(layer "B.Fab")
@@
 			)
 		)
-		(property "Value" "33E"
+		(property "Value" "2-2.2M (33E)"
 			(at 0 -1 0)
 			(layer "B.Fab")
@@
 			)
 		)
-		(property "Value" "33E"
+		(property "Value" "2-2.2M (33E)"
 			(at 0 -1 0)
 			(layer "B.Fab")
@@
 			)
 		)
-		(property "Value" "33E"
+		(property "Value" "2-2.2M (33E)"
 			(at 0 -1 0)
 			(layer "B.Fab")
@@
 			)
 		)
-		(property "Value" "33E"
+		(property "Value" "2-2.2M (33E)"
 			(at 0 -1 0)
 			(layer "B.Fab")
@@
 			)
 		)
-		(property "Value" "33E"
+		(property "Value" "2-2.2M (33E)"
 			(at 0 -1 0)
 			(layer "B.Fab")
