File: kiss-masterboard/masterboard_v0.2/kiss-masterboard.kicad_pcb (KiCad board)
At the start: 4 copper layers, 187 x 152 mm, 172 parts, among them J1 Cubebatt_host, J10 CRESET, J11 Jumper, J12 Jumper, J13 Conn_02x08_Odd_Even, J14 Conn_02x08_Odd_Even, J15 jmp, J16 jmp, J17 Conn_02x05_Counter_Clockwise, J18 Conn_02x02_Counter_Clockwise, J2 Conn_01x02, J3 Conn_01x02, J4 Conn_01x02, J5 Conn_01x02, J6 Conn_01x02, J7 Conn_01x02, J8 Jumper, J9 Conn_01x07_Pin, P2 CONN_02X20, U10 CSD86360Q5D, U11 TLV75733PDBV, U13 SN74LVC8T245, U14 W25Q, U17 12MHz, U2 SN74LVC8T245, U3 TPS56339DDC, U4 ICE40UP5k-SG48, U5 SN74LVC8T245, U7 SPH0645LM4H, U8 TLV75709PDBV, U9 TPS53819A

Commit message: replace 2.2mohm with 33ohm for all hub75
Parts:
- D5: value GRN -> LED, green
- D6: value BLU -> LED, blue
- J17: value Conn_02x05_Counter_Clockwise -> Conn_02x06_Counter_Clockwise
- R11: value 10k %% -> 10K 1%
- R15, R16, R17, R21, R22, R23, R26, R27, R30: value 10k -> 10K 1%
- R51, R52, R53, R54, R55, R56, R57, R58, R59, R60, R61, R62, R63, R64, R65, R66, R67, R68, R69, R70, R71, R72, R73, R74, R75, R76, R77, R78: value 2-2.2M (33E) -> 33R
